File: pcb_hardware/dmf_relay_board/_autosave-dmf_relay_board.kicad_pcb (KiCad board)
At the start: 2 copper layers, 100 x 96.5 mm, 70 parts, among them J1 HVPS, J2 Relays to Electrodes 1, J3 Relays to Electrodes 2, J4 Electrodes from Relay 1, J5 Electrodes from Relay 2, U1 HV507

Commit message: electrode footprints placed - routing now
Connections:
- J4 pad 1: Net-(EXS1-Pad1) -> Net-(J4-Pad1)
- J4 pad 10: Net-(EXS10-Pad1) -> Net-(J4-Pad10)
- J4 pad 11: Net-(EXS11-Pad1) -> Net-(J4-Pad11)
- J4 pad 12: Net-(EXS12-Pad1) -> Net-(J4-Pad12)
- J4 pad 13: Net-(EXS13-Pad1) -> Net-(J4-Pad13)
- J4 pad 14: Net-(EXS14-Pad1) -> Net-(J4-Pad14)
- J4 pad 15: Net-(EXS15-Pad1) -> Net-(J4-Pad15)
- J4 pad 16: Net-(EXS16-Pad1) -> Net-(J4-Pad16)
- J4 pad 17: Net-(EXS17-Pad1) -> Net-(J4-Pad17)
- J4 pad 18: Net-(EXS18-Pad1) -> Net-(J4-Pad18)
- J4 pad 19: Net-(EXS19-Pad1) -> Net-(J4-Pad19)
- J4 pad 2: Net-(EXS2-Pad1) -> Net-(J4-Pad2)
- J4 pad 20: Net-(EXS20-Pad1) -> Net-(J4-Pad20)
- J4 pad 21: Net-(EXS21-Pad1) -> Net-(J4-Pad21)
- J4 pad 22: Net-(EXS22-Pad1) -> Net-(ELG6-Pad1)
- J4 pad 23: Net-(EXS23-Pad1) -> Net-(J4-Pad23)
- J4 pad 24: Net-(EXS24-Pad1) -> Net-(ELG5-Pad1)
- J4 pad 25: Net-(ESM1-Pad1) -> Net-(J4-Pad25)
- J4 pad 26: Net-(ESM2-Pad1) -> Net-(ESM30-Pad1)
- J4 pad 27: Net-(ESM3-Pad1) -> Net-(J4-Pad27)
- J4 pad 28: Net-(ESM4-Pad1) -> Net-(ESM29-Pad1)
- J4 pad 29: Net-(ESM5-Pad1) -> Net-(J4-Pad29)
- J4 pad 3: Net-(EXS3-Pad1) -> Net-(J4-Pad3)
- J4 pad 30: Net-(ESM6-Pad1) -> Net-(ESM28-Pad1)
- J4 pad 4: Net-(EXS4-Pad1) -> Net-(J4-Pad4)
- J4 pad 5: Net-(EXS5-Pad1) -> Net-(J4-Pad5)
- J4 pad 6: Net-(EXS6-Pad1) -> Net-(J4-Pad6)
- J4 pad 7: Net-(EXS7-Pad1) -> Net-(J4-Pad7)
- J4 pad 8: Net-(EXS8-Pad1) -> Net-(J4-Pad8)
- J4 pad 9: Net-(EXS9-Pad1) -> Net-(J4-Pad9)
- J5 pad 1: Net-(ESM7-Pad1) -> Net-(J5-Pad1)
- J5 pad 10: Net-(ESM16-Pad1) -> Net-(EXS23-Pad1)
- J5 pad 11: Net-(ESM17-Pad1) -> Net-(J5-Pad11)
- J5 pad 12: Net-(ESM18-Pad1) -> Net-(EXS22-Pad1)
- J5 pad 13: Net-(ESM19-Pad1) -> Net-(J5-Pad13)
- J5 pad 14: Net-(ESM20-Pad1) -> Net-(EXS21-Pad1)
- J5 pad 15: Net-(ESM21-Pad1) -> Net-(J5-Pad15)
- J5 pad 16: Net-(ESM22-Pad1) -> Net-(J5-Pad16)
- J5 pad 17: Net-(ESM23-Pad1) -> Net-(J5-Pad17)
- J5 pad 18: Net-(ESM24-Pad1) -> Net-(EXS14-Pad1)
- J5 pad 19: Net-(ESM25-Pad1) -> Net-(J5-Pad19)
- J5 pad 2: Net-(ESM8-Pad1) -> Net-(ESM27-Pad1)
- J5 pad 20: Net-(ESM26-Pad1) -> Net-(ESM14-Pad1)
- J5 pad 21: Net-(ESM27-Pad1) -> Net-(J5-Pad21)
- J5 pad 22: Net-(ESM28-Pad1) -> Net-(J5-Pad22)
- J5 pad 23: Net-(ESM29-Pad1) -> Net-(J5-Pad23)
- J5 pad 24: Net-(ESM30-Pad1) -> Net-(J5-Pad24)
- J5 pad 25: Net-(ELG1-Pad1) -> Net-(J5-Pad25)
- J5 pad 26: Net-(ELG2-Pad1) -> Net-(J5-Pad26)
- J5 pad 27: Net-(ELG3-Pad1) -> Net-(J5-Pad27)
- J5 pad 28: Net-(ELG4-Pad1) -> Net-(J5-Pad28)
- J5 pad 29: Net-(ELG5-Pad1) -> Net-(J5-Pad29)
- J5 pad 3: Net-(ESM9-Pad1) -> Net-(J5-Pad3)
- J5 pad 30: Net-(ELG6-Pad1) -> Net-(J5-Pad30)
- J5 pad 4: Net-(ESM10-Pad1) -> Net-(ESM26-Pad1)
- J5 pad 5: Net-(ESM11-Pad1) -> Net-(J5-Pad5)
- J5 pad 6: Net-(ESM12-Pad1) -> Net-(ESM25-Pad1)
- J5 pad 7: Net-(ESM13-Pad1) -> Net-(J5-Pad7)
- J5 pad 8: Net-(ESM14-Pad1) -> Net-(EXS24-Pad1)
- J5 pad 9: Net-(ESM15-Pad1) -> Net-(J5-Pad9)
