File: pcb_hardware/dmf_relay_board/dmf_relay_board.kicad_pcb (KiCad board)
At the start: 4 copper layers, 100 x 96.5 mm, 76 parts, among them J1 HVPS, J2 Relays to Electrodes 1, J3 Relays to Electrodes 2, J4 Electrodes from Relay 1, J5 Electrodes from Relay 2, M1 MountingHole_3.2mm_M3, M2 MountingHole_3.2mm_M3, M3 MountingHole_3.2mm_M3, M4 MountingHole_3.2mm_M3, M5 MountingHole_3.2mm_M3, M6 MountingHole_3.2mm_M3, U1 HV507

Commit message: final fab files added
Routing:
- net GND: track 50.6 -> 21.1 mm
- net CHNL_13: track 70.4 -> 65.8 mm
- net CHNL_12: track 69.8 -> 65.5 mm
- net CHNL_11: track 67.7 -> 63.6 mm
- net CHNL_10: track 67.6 -> 63.6 mm
- net CHNL_9: track 51.2 -> 47.9 mm
- net CHNL_8: track 58.7 -> 56.0 mm
- net CHNL_7: track 62.5 -> 59.9 mm
- net CHNL_6: track 67.1 -> 65.0 mm
- net CHNL_5: track 70.3 -> 68.7 mm
- net CHNL_3: track 78.1 -> 77.1 mm
- net CHNL_4: track 74.4 -> 73.5 mm
- net DI: track 53.8 -> 53.1 mm
